File: schematic/pslab-mini.kicad_sch (KiCad schematic)
At the start: 0 parts

Commit message: Update pslab-mini.kicad_sch
Other:
- title: PSLab-Mini -> PSLab-Mini-T4-1
Changed lines of the file:
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@@
 	(paper "A4")
 	(title_block
-		(title "PSLab-Mini")
+		(title "PSLab-Mini-T4-1")
 		(date "2025-07-16")
 		(rev "0.0.0")

Commit message: Update pslab-mini.kicad_sch
Other:
- title: PSLab-Mini-T4-1 -> PSLab-Mini-T4-2
Changed lines of the file:
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@@
 	(paper "A4")
 	(title_block
-		(title "PSLab-Mini-T4-1")
+		(title "PSLab-Mini-T4-2")
 		(date "2025-07-16")
 		(rev "0.0.0")
