File: schematic/pslab-mini.kicad_sch (KiCad schematic)
At the start: 182 parts, among them J1 USB_C_Receptacle_USB2.0_16P, J2 BAT, J3 Conn_Coaxial, J4 Conn_Coaxial, J5 Conn_02x16_Odd_Even, J6 Conn_01x15_Socket, J7 Conn_02x03_Top_Bottom, Q1 MMBT3904, Q2 MMBT3904, SW1 Reset, SW4 Power, U1 AMS1117-3.3, U10 OPA356AIDBVR, U11 ESP32-C3, U12 W25Q32JV, U2 MT2496, U3 IP5189T, U4 SP0503BAHT, U5 OPA356AIDBVR, U6 OPA356AIDBVR, U7 TLV9001IDCK, U8 STM32H563RIT6, U9 OPA356AIDBVR, X1 32kHz768, Y1 Crystal_25MHz, Y2 40MHz

Commit message: init: updated KiCAD version and initial settings
Other:
- title: PSLab-Mini -> PSLab-Mini-RP2350
Changed lines of the file:
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@@
 (kicad_sch
-	(version 20250114)
+	(version 20260306)
 	(generator "eeschema")
-	(generator_version "9.0")
-	(paper "User" 477.52 350)
+	(generator_version "10.0")
+	(paper "User" 477.52 350.0000112)
 	(title_block
-		(title "PSLab-Mini")
-		(date "2025-07-16")
-		(rev "0.0.0")
+		(title "PSLab-Mini-RP2350")
+		(date "2026-08-24")
+		(rev "1.0.0")
 	)
